Commit message: URDFs edited to handle multi-links. Example added.(cherry-pick of kinetic branch)

File: urdf/rs200_simulation.xacro (robot description, xacro)
@@ -5,10 +5,16 @@
 -->
 <robot name="robot_with_rs200" xmlns:xacro="http://ros.org/wiki/xacro">
-    <link name="world"/>
     <!-- Import macro for realsense-RS200 camera-->
     <xacro:include filename="$(find realsense_gazebo_plugin)/urdf/realsense-RS200.macro.xacro"/>
     <!-- Create camera instance -->
-    <xacro:realsense-rs200 prefix="" parent="world">
-        <origin xyz="0 0 1.0" rpy="0 0 0" />
-    </xacro:realsense-rs200>
+    <xacro:realsense-rs200/>
+    <!-- Gazebo world link required to position the robot with respect to origin -->
+    <!-- the name "world" is mandatory for Gazebo! -->
+    <link name="world"/>
+    <!-- Place camera referenced to world frame -->
+    <joint name="realsense_joint" type="fixed">
+        <parent link="world"/>
+        <child link="rs200_camera"/>
+        <origin rpy="0 0 0" xyz="0 0 1.0"/>
+    </joint>
 </robot>

Commit message: minor

File: urdf/rs200_simulation.xacro (robot description, xacro)
@@ -5,5 +5,4 @@
 -->
 <robot name="robot_with_rs200" xmlns:xacro="http://ros.org/wiki/xacro">
-    <link name="world"/>
     <!-- Import macro for realsense-RS200 camera-->
     <xacro:include filename="$(find realsense_gazebo_plugin)/urdf/realsense-RS200.macro.xacro"/>
