Commit message: URDFs edited to handle multi-links. Example added.(cherry-pick of kinetic branch)

File: urdf/realsense-RS200.macro.xacro (robot description, xacro)
@@ -9,9 +9,12 @@
             * Virtual depth coordinate frame
         Configured to work with Gazebo if desired.
+    Update of Maik93: in order to handle camera positions while attaching the Realsense to other links,
+    optional parameters "parent_link, origin_x, origin_y, origin_z" are implemented.
+    See urdf/rs200_simulation_multilink.xacro for details.
 -->
 <robot xmlns:xacro="http://ros.org/wiki/xacro">
-<xacro:macro name="realsense-rs200" params="prefix parent *origin">
+<xacro:macro name="realsense-rs200" params="parent_link:='rs200_camera' origin_x:=0 origin_y:=0 origin_z:=0">
     <!-- Camera link -->
-    <link name="${prefix}rs200_camera">
+    <link name="rs200_camera">
         <visual>
             <origin rpy="0 0 0" xyz="0 0 0"/>
@@ -37,36 +40,30 @@
         </inertial>
     </link>
-    <!-- Connect camera to parent frame-->
-    <joint name="${prefix}realsense_joint" type="fixed">
-        <parent link="${parent}"/>
-        <child link="${prefix}rs200_camera"/>
-        <xacro:insert_block name="origin"/>
-    </joint>
     <!-- Virtual links representing the cameras positons and orientations-->
-    <link name="${prefix}color" />
-    <link name="${prefix}depth" />
-    <link name="${prefix}ired1" />
-    <link name="${prefix}ired2" />
+    <link name="color" />
+    <link name="depth" />
+    <link name="ired1" />
+    <link name="ired2" />
     <!-- Joints positioning the virtual links with respect to the camera main link-->
-    <joint name="${prefix}color_joint" type="fixed">
-        <parent link="${prefix}rs200_camera" />
-        <child link="${prefix}color" />
+    <joint name="color_joint" type="fixed">
+        <parent link="rs200_camera" />
+        <child link="color" />
         <!-- <origin xyz="0 -0.046 0.004" rpy="0 0 0"/> -->
-        <!-- The default position is change since in Rviz the cloud depth axis is Z not X-->
+        <!-- The default position is changed since in Rviz the cloud depth axis is Z not X-->
         <origin xyz="0 -0.046 0.004" rpy="${pi/2} ${pi} ${pi/2}"/>
     </joint>
-    <joint name="${prefix}depth_joint" type="fixed">
-        <parent link="${prefix}rs200_camera" />
-        <child link="${prefix}depth" />
+    <joint name="depth_joint" type="fixed">
+        <parent link="rs200_camera" />
+        <child link="depth" />
         <origin xyz="0 -0.03 0.004" rpy="0 0 0"/>
     </joint>
-    <joint name="${prefix}ired1_joint" type="fixed">
-        <parent link="${prefix}rs200_camera" />
-        <child link="${prefix}ired1" />
+    <joint name="ired1_joint" type="fixed">
+        <parent link="rs200_camera" />
+        <child link="ired1" />
         <origin xyz="0 -0.06 0.004" rpy="0 0 0"/>
     </joint>
-    <joint name="${prefix}ired2_joint" type="fixed">
-        <parent link="${prefix}rs200_camera" />
-        <child link="${prefix}ired2" />
+    <joint name="ired2_joint" type="fixed">
+        <parent link="rs200_camera" />
+        <child link="ired2" />
         <origin xyz="0 0.01 0.004" rpy="0 0 0"/>
     </joint>
@@ -79,5 +76,5 @@
     </gazebo>
     <!-- Load parameters to model's main link-->
-    <gazebo reference="${prefix}rs200_camera">
+    <gazebo reference="${parent_link}">
         <self_collide>0</self_collide>
         <enable_wind>0</enable_wind>
@@ -94,6 +91,6 @@
         <min_depth>0</min_depth>-->
         <sensor name="color" type="camera">
-            <pose frame="">0 -0.046 0.004 0 0 0</pose>
-            <camera name="${prefix}rs200_camera">
+            <pose frame="">${origin_x + 0} ${origin_y - 0.046} ${origin_z + 0.004} 0 0 0</pose>
+            <camera name="__default__">
             <horizontal_fov>1.047</horizontal_fov>
             <image>
@@ -117,6 +114,6 @@
         </sensor>
         <sensor name="ired1" type="camera">
-            <pose frame="">0 -0.06 0.004 0 0 0</pose>
-            <camera name="${prefix}rs200_camera">
+            <pose frame="">${origin_x + 0} ${origin_y - 0.06} ${origin_z + 0.004} 0 0 0</pose>
+            <camera name="__default__">
             <horizontal_fov>1.047</horizontal_fov>
             <image>
@@ -140,6 +137,6 @@
         </sensor>
         <sensor name="ired2" type="camera">
-            <pose frame="">0 0.01 0.004 0 0 0</pose>
-            <camera name="${prefix}rs200_camera">
+            <pose frame="">${origin_x + 0} ${origin_y + 0.01} ${origin_z + 0.004} 0 0 0</pose>
+            <camera name="__default__">
             <horizontal_fov>1.047</horizontal_fov>
             <image>
@@ -163,6 +160,6 @@
         </sensor>
         <sensor name="depth" type="depth">
-            <pose frame="">0 -0.03 0.004 0 0 0</pose>
-            <camera name="${prefix}rs200_camera">
+            <pose frame="">${origin_x + 0} ${origin_y - 0.03} ${origin_z + 0.004} 0 0 0</pose>
+            <camera name="__default__">
             <horizontal_fov>1.047</horizontal_fov>
             <image>

File: urdf/rs200_simulation.xacro (robot description, xacro)
@@ -9,6 +9,13 @@
     <xacro:include filename="$(find realsense_gazebo_plugin)/urdf/realsense-RS200.macro.xacro"/>
     <!-- Create camera instance -->
-    <xacro:realsense-rs200 prefix="" parent="world">
-        <origin xyz="0 0 1.0" rpy="0 0 0" />
-    </xacro:realsense-rs200>
+    <xacro:realsense-rs200/>
+    <!-- Gazebo world link required to position the robot with respect to origin -->
+    <!-- the name "world" is mandatory for Gazebo! -->
+    <link name="world"/>
+    <!-- Place camera referenced to world frame -->
+    <joint name="realsense_joint" type="fixed">
+        <parent link="world"/>
+        <child link="rs200_camera"/>
+        <origin rpy="0 0 0" xyz="0 0 1.0"/>
+    </joint>
 </robot>

Commit message: DAE model rescaled to fix wrong sizes in RViz

File: urdf/realsense-RS200.macro.xacro (robot description, xacro)
@@ -20,5 +20,5 @@
             <origin rpy="0 0 0" xyz="0 0 0"/>
             <geometry>
-                <mesh filename="package://realsense_gazebo_plugin/models/realsense_camera/meshes/realsense.dae"/>
+                <mesh filename="package://realsense_gazebo_plugin/models/realsense_camera/meshes/realsense.dae" scale="0.01 0.01 0.01"/>
             </geometry>
         </visual>

Commit message: real image dimensions, Hz and topic names

File: urdf/realsense-RS200.macro.xacro (robot description, xacro)
@@ -14,7 +14,7 @@
 -->
 <robot xmlns:xacro="http://ros.org/wiki/xacro">
-<xacro:macro name="realsense-rs200" params="parent_link:='rs200_camera' origin_x:=0 origin_y:=0 origin_z:=0">
+<xacro:macro name="realsense-rs200" params="parent_link:='camera_link' origin_x:=0 origin_y:=0 origin_z:=0">
     <!-- Camera link -->
-    <link name="rs200_camera">
+    <link name="camera_link">
         <visual>
             <origin rpy="0 0 0" xyz="0 0 0"/>
@@ -47,5 +47,5 @@
     <!-- Joints positioning the virtual links with respect to the camera main link-->
     <joint name="color_joint" type="fixed">
-        <parent link="rs200_camera" />
+        <parent link="camera_link" />
         <child link="color" />
         <!-- <origin xyz="0 -0.046 0.004" rpy="0 0 0"/> -->
@@ -54,15 +54,15 @@
     </joint>
     <joint name="depth_joint" type="fixed">
-        <parent link="rs200_camera" />
+        <parent link="camera_link" />
         <child link="depth" />
         <origin xyz="0 -0.03 0.004" rpy="0 0 0"/>
     </joint>
     <joint name="ired1_joint" type="fixed">
-        <parent link="rs200_camera" />
+        <parent link="camera_link" />
         <child link="ired1" />
         <origin xyz="0 -0.06 0.004" rpy="0 0 0"/>
     </joint>
     <joint name="ired2_joint" type="fixed">
-        <parent link="rs200_camera" />
+        <parent link="camera_link" />
         <child link="ired2" />
         <origin xyz="0 0.01 0.004" rpy="0 0 0"/>
@@ -110,5 +110,5 @@
             </camera>
             <always_on>1</always_on>
-            <update_rate>60</update_rate>
+            <update_rate>30</update_rate>
             <visualize>1</visualize>
         </sensor>
@@ -118,6 +118,6 @@
             <horizontal_fov>1.047</horizontal_fov>
             <image>
-                <width>640</width>
-                <height>480</height>
+                <width>480</width>
+                <height>360</height>
                 <format>L_INT8</format>
             </image>
@@ -133,5 +133,5 @@
             </camera>
             <always_on>1</always_on>
-            <update_rate>60</update_rate>
+            <update_rate>30</update_rate>
             <visualize>0</visualize>
         </sensor>
@@ -141,6 +141,6 @@
             <horizontal_fov>1.047</horizontal_fov>
             <image>
-                <width>640</width>
-                <height>480</height>
+                <width>480</width>
+                <height>360</height>
                 <format>L_INT8</format>
             </image>
@@ -156,5 +156,5 @@
             </camera>
             <always_on>1</always_on>
-            <update_rate>60</update_rate>
+            <update_rate>30</update_rate>
             <visualize>0</visualize>
         </sensor>
@@ -164,6 +164,6 @@
             <horizontal_fov>1.047</horizontal_fov>
             <image>
-                    <width>640</width>
-                    <height>480</height>
+                    <width>480</width>
+                    <height>360</height>
             </image>
             <clip>
@@ -178,5 +178,5 @@
             </camera>
             <always_on>1</always_on>
-            <update_rate>60</update_rate>
+            <update_rate>30</update_rate>
             <visualize>0</visualize>
         </sensor>

File: urdf/rs200_simulation.xacro (robot description, xacro)
@@ -15,5 +15,5 @@
     <joint name="realsense_joint" type="fixed">
         <parent link="world"/>
-        <child link="rs200_camera"/>
+        <child link="camera_link"/>
         <origin rpy="0 0 0" xyz="0 0 1.0"/>
     </joint>

File: urdf/rs200_simulation_multilink.xacro (robot description, xacro)
@@ -36,5 +36,5 @@
     <joint name="realsense_joint" type="fixed">
         <parent link="box"/>
-        <child link="rs200_camera"/>
+        <child link="camera_link"/>
         <origin rpy="0 0 0" xyz="0 0 0.2"/>
     </joint>
